File: PCB/ModuloComunicacionesPCB/Schematic_Sensing_Module.sch (EAGLE design)
At the start: 63 parts, among them IC1 MCP3202P, Q1 CSM-7X-DU, SW2 1825910-6, U1 ATMEGA328P-PU, U2 LP38690DT-5.0, U2_VCC NCP699SN33T1G, U3_VDD NCP699SN33T1G

Commit message: avance en esquematico para la PCB
Parts:
- removed ACS_PIN: (no value), pinhead:PINHD-1X3
- removed IC1: MCP3202P, microchip:MCP3202P
- removed MCP_1: MCP6002-I/MS, MCP6002-I_MS-2:MCP6002-I/MS
- removed MCP_2, MCP_3, MCP_4: MCP6002-I/MS, MCP6002-I_MS:MCP6002-I/MS
- removed R18: 15k, resistor:R-US_R0805
- removed R20: 1.5k, rcl:R-US_R1206
- removed R21, R24, R25, R26: 10k, rcl:R-US_R1206
- removed R23: 560, rcl:R-US_R1206
- removed R27: 22k, rcl:R-US_R1206
- removed TEMP_PIN: (no value), con-lstb:MA04-1
- removed TR_TRG0: 20k, rcl:R-TRIMM64W
- removed TR_TRG1: 20K, rcl:R-TRIMM64W
- removed U2_VCC, U3_VDD: NCP699SN33T1G, NCP699SN33T1G:NCP699SN33T1G
- removed WATER_PIN: (no value), con-lstb:MA03-1
- added Q2: MMBT2222A, MMBT2222A:MMBT2222A
- added R10: 4.7k, rcl:R-EU_M1206
- added R11: 75k, rcl:R-EU_R1206
- added R12: 1.43Meg, rcl:R-EU_R0805
- added R13, R14: 91, rcl:R-EU_R1206
- added R15, R16, R17, R4, R5: 0.1, rcl:R-EU_R1206
- added R6: 10, rcl:R-EU_R0805
- added R9: 10k, rcl:R-EU_R0805
- added U$3: MCP6002-E/MS, MCP6002-E_MS:MCP6002-E/MS
- added U$5: MCP33121, mcp33121:MCP33121
- added U$6: TERMINAL-TB2, TERMINAL-TB001:TERMINAL-TB2
- added U$7: REF3450, SOT95P280X145-6N:REF3450
- added U3: MCP1501T-18E/SN, MCP1501T-18E_SN:MCP1501T-18E/SN
- added U4: ACS723LLCTR-05AB-T, ACS723LLCTR-05AB-T:ACS723LLCTR-05AB-T
- added U5: OPA320AIDBVR, OPA320AIDBVR:OPA320AIDBVR
- C10: value 10n -> 1nF; device rcl:C-EUC0805 -> rcl:C-EUC1206
- C13: value (none) -> 620pF; device rcl:C-USC0805 -> rcl:C-EUC1206
- C14, C15, C21: value 0.1u -> 100n; device rcl:C-EUC0805 -> rcl:C-EUC1206
- C16: value 1u -> 100nF; device rcl:C-EUC0805 -> rcl:C-EUC1206
- C18: value 0.1u -> 1uF; device rcl:C-EUC0805 -> rcl:C-EUC1206
- C19: value 0.1u -> 10uF; device rcl:C-EUC0805 -> rcl:C-EUC1206
- C2, C3: value (none) -> 1uF; device rcl:C-USC0805 -> rcl:C-EUC1206
- C20: value 1u -> 100n; device rcl:C-EUC0805 -> rcl:C-EUC1206
- C23, C5: value 0.1u -> 1u; device rcl:C-EUC0805 -> rcl:C-EUC1206
- C4: value (none) -> 2.2uF; device rcl:C-USC0805 -> rcl:C-EUC1206
- C6: value 10n -> 1u; device rcl:C-EUC0805 -> rcl:C-EUC1206
- C7, C8: value 10n -> 2.2uF; device rcl:C-EUC0805 -> T491A106K010AT7280:T491A106K010AT7280
- C9: value 10n -> 100pF; device rcl:C-EUC0805 -> rcl:C-EUC1206
- R1: value 560 -> 4.7k; device rcl:R-US_R1206 -> rcl:R-EU_R1206
- R3: value 1.5k -> 0.1; device rcl:R-US_R1206 -> rcl:R-EU_R1206
- U2: value LP38690DT-5.0 -> LP38692MP-5.0; device LP38690DT-5.0:LP38690DT-5.0 -> LP38692MP-5.0:LP38692MP-5.0
Connections:
- removed net B+: U$4.VIN1+
- removed net DWS: C20.1, MCP_4.VINA+, R23.2, WATER_PIN.2
- removed net VBTR: C16.2, MCP_3.VINB+, R18.2
- removed net VCC33: C15.2, C18.1, C19.1, C3.1, MCP_4.VDD, R20.2, R3.2, TEMP_PIN.1, U$4.VCC, U2_VCC.VOUT, WATER_PIN.1
- removed net VINA+_MCP_2: C7.1, MCP_2.VINA+, R27.2
- removed net VINADC0: C6.1, C9.1, IC1.CH0, MCP_2.VINB-, MCP_2.VOUTB
- removed net VINADC1: IC1.CH1, MCP_3.VINB-, MCP_3.VOUTB
- removed net VINB+_MCP_1: MCP_1.VINB+, R25.1, R26.1
- removed net VINB+_MCP_2: C10.2, MCP_2.VINB+, R21.1
- removed net VINB-_MCP_1: MCP_1.VINB-, R24.1, TR_TRG0.A
- removed net VIN_CURR: ACS_PIN.2, MCP_1.VINA+
- removed net VOA: MCP_1.VINA-, MCP_1.VOUTA, R24.2
- removed net VOATR: MCP_3.VINA-, MCP_3.VOUTA, R18.1
- removed net VOA_MCP_2: MCP_2.VINA-, MCP_2.VOUTA, R1.2
- removed net VOB: MCP_1.VOUTB, R27.1, TR_TRG0.S
- removed net VTR: C14.1, MCP_3.VINA+, TR_TRG1.S
- new net N$1: R3.2, U$2.GNDF
- new net N$10: U$6.1, U4.IP+
- new net N$11: U$6.2, U4.IP-
- new net N$12: R11.2, U4.VIOUT
- new net N$14: C10.2, R11.1, R12.1
- new net N$15: C10.1, R13.1, U5.-IN, U5.OUT
- new net N$16: C13.2, R13.2, U$5.IN+
- new net N$17: C13.1, R14.2, U$5.IN-
- new net N$18: R16.2, U$7.OUTF
- new net N$19: R17.2, U$7.OUTS
- new net N$2: C4.1, Q2.B, R1.2
- new net N$20: R15.2, U$7.GNDF
- new net N$6: R5.2, U$2.OUTS
- new net N$7: R6.2, R9.2, U3.FEEDBACK, U3.OUT
- new net N$8: R10.1, U4.BW_SEL
- new net VACS: C15.1, C23.1, R10.2, R16.1, R17.1, U4.VCC
- new net VLP5: C19.2, C20.1, C3.1, U$5.DVIO, U2.VOUT
- new net VOREG: C5.1, Q2.E, U$2.EN, U$2.IN, U$7.EN, U$7.IN
- new net VREF18: C21.2, C8.1, R6.1, U$5.AVDD
- new net VREF5: C14.2, C16.1, C18.1, C6.1, C7.1, R4.1, R5.1, U$5.VREF, U3.!SHDN, U3.VDD, U5.V+
- net +5V: no longer ACS_PIN.3, C21.1, C23.1, C5.1, IC1.VDD/VREF, MCP_1.VDD, MCP_2.VDD, MCP_3.VDD, R25.2, TR_TRG1.E, U2_VCC.EN, U2_VCC.VIN, U3_VDD.EN, U3_VDD.VIN
- net A0: no longer MCP_4.VINA-, MCP_4.VOUTA
- net AMISO: now also U$5.SDO; no longer IC1.DOUT
- net AMOSI: now also U$5.SDI; no longer IC1.DIN
- net ASCK: now also U$5.CLK; no longer IC1.CLK
- net ASS: now also U$5.CNVST; no longer IC1.!CS!/SHDN
- net B-INA: no longer U$4.VIN1-
- net GND: now also C14.1, C15.2, C16.2, C19.1, C21.1, C6.2, C7.2, C9.2, R14.1, R15.1, R3.1, R9.1, U$2.GNDS, U$5.GND, U$7.GNDS, U2.GND, U3.GND, U4.GND, U5.V-; no longer ACS_PIN.1, C10.1, C13.2, C14.2, C15.1, C16.1, C19.2, C21.2, IC1.VSS, MCP_1.VSS, MCP_2.VSS, MCP_3.VSS, MCP_4.VINB+, MCP_4.VINB-, MCP_4.VSS, R23.1, R26.2, TEMP_PIN.2, TR_TRG1.A, U$4.GND, U2_VCC.GND, U3_VDD.GND, WATER_PIN.3
- net N$13: now also C9.1, R12.2, U5.+IN; no longer C6.2, C9.2, R1.1, R21.2
- net N$5: now also R4.2, U$2.OUTF; no longer C7.2, C8.1
- net SCL: no longer R3.1, TEMP_PIN.3, U$4.SCL
- net SDA: no longer R20.1, TEMP_PIN.4, U$4.SDA
- net VDD33: no longer C4.1, U3_VDD.VOUT
- net VSUPPLY: now also Q2.C, R1.1, U2.VEN, U2.VIN; no longer C13.1
Other:
- note added: "1206 10V"
- note added: "ALIMENTACION 5V MIX"
- note added: "ALIMENTACION 5V+"
- note added: "ALIMENTACION CIRCUITOS ADC"
- note removed: "ANALOG SUPPLY 3.3v"
- note removed: "DIGITAL SUPPLY 3.3v"
- note removed: "TRIGGER"
- note removed: "cap 0805"
- moved on the sheet: C1, C10, C11, C12, C13, C14, C15, C16, C18, C19, C2, C20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

Commit message: terminacion de esquematico e inicio del esquematico del coordinador
Parts:
- removed XB1: XBEE-PRO, maxstream:XBEE-PRO
- added C25, C26, C27, C28, C29, C30, C31, C32: 0.1uF, rcl:C-EUC1206
- added C33: 1nF, rcl:C-EUC1206
- added C34: 2.2uF, rcl:C-EUC1206
- added J1, J2, J3, J4: TERMINAL-TB3, TERMINAL-TB001:TERMINAL-TB3
- added R18, R19: 560, rcl:R-EU_R1206
- added U$8: XBEE_REG_MODULE, XBEE_REG:XBEE_REG_MODULE
- C11, C12: value 22p -> 22pF; device rcl:C-USC1206 -> rcl:C-EUC0805
- C14, C15, C20, C21: value 100n -> 100nF
- C17: value 8.2pF -> 18pF
- C2, C3: value 1uF -> 2.2uF
- C22: value 0.1u -> 0.1uF
Connections:
- removed net A0: U1.PC0
- removed net A1: U1.PC1
- removed net A2: U1.PC2
- removed net A3: U1.PC3
- new net DATAT1: C27.1, J3.2, U1.PD6
- new net DATAT2: C28.1, J4.2, U1.PD7
- new net DATAW1: C25.1, J1.3, R19.1, U$3.VINA+
- new net DATAW2: C26.1, J2.3, R18.1, U$3.VINB+
- new net VOW1: U$3.VINA-, U$3.VOUTA, U1.PC0
- new net VOW2: U$3.VINB-, U$3.VOUTB, U1.PC1
- net +5V: no longer C22.1, D1.C, R2.2, U1.AVCC, U1.VCC
- net B+INA: now also U$4.VIN-
- net B-INA: now also U$4.VIN+
- net BATH: now also U1.PB0; no longer U1.PD6
- net BATL: now also U1.PB1; no longer U1.PD5
- net GND: now also C25.2, C26.2, C27.2, C28.2, C29.2, C30.2, C31.2, C32.2, C33.2, C34.1, J1.1, J2.1, J3.3, J4.3, R18.2, R19.2, U$3.VSS, U$4.GND, U$8.GND, U$8.GND1, U$8.GND2, U$8.GND3; no longer XB1.GND
- net N$12: now also C33.1
- net OSC+: now also C12.1; no longer C11.1
- net OSC-: now also C11.1; no longer C12.1
- net RX1: now also U$8.TX; no longer XB1.DOUT
- net SCL: now also U$4.SCL
- net SDA: now also U$4.SDA
- net TX1: now also U$8.RX; no longer XB1.DIN/!CONFIG
- net VDD33: now also C29.1, U$4.VCC, U$8.3.3V, U$8.3.3V1; no longer C17.1, C24.1, XB1.VCC
- net VLP5: now also C22.1, C30.1, C31.1, C32.1, C34.2, D1.C, J1.2, J2.2, J3.1, J4.1, R2.2, U$3.VDD, U1.AVCC, U1.VCC
- net VOUT+: now also C17.1, C24.1
Other:
- note added: "1206 TA"
- note added: "1206 inamovible"
- note added: "ALIMENTACION 1.8 AVCC"
- note added: "ALIMENTACION 5V+ MIX"
- note removed: "12206"
- note removed: "ALIMENTACION 5V MIX"
- note removed: "ALIMENTACION 5V+"
- note removed: "INA"
- note removed: "must be less than 10k"
- moved on the sheet: C1, C10, C11, C12, C13, C14, C15, C16, C17, C18, C19, C20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

Commit message: avances en placing de la pcb del transmisor
Parts:
- removed BAT_PIN: (no value), pinhead:PINHD-1X2
- removed C24: (no value), rcl:C-USC0805
- removed FTDI_PIN: (no value), pinhead:PINHD-1X4
- removed R15, R16, R17, R3, R4, R5: 0.1, rcl:R-EU_R1206
- added C35: 2.2uF, rcl:C-EUC1206
- added JP1: (no value), pinhead:PINHD-1X4/90
- C2, C3: value 2.2uF -> cambiar por los de 10uF ceramicos de didacticas
- U$4: value INA219_BB -> INABB; device INA219_BB:INA219_BB -> INA219BB:INABB
- renumbered J1 to WS1, J2 to WS2, J3 to TS1, J4 to TS2, Q2 to 2N2222, U$2 to R3450, U$3 to MCP6002, U$6 to IACT, U$7 to REF3450, U2 to LP38692, U4 to ACS723, U5 to OPA320
Connections:
- net N$10 renamed IP+
- net N$11 renamed IP-
- net N$12 renamed VO
- net N$13 renamed VIN+
- net N$15 renamed VIN-
- net N$8 renamed BWSEL
- removed net +5V: U$1.IN+
- removed net N$1: R3.2, R3450.GNDF
- removed net N$18: R16.2, REF3450.OUTF
- removed net N$19: R17.2, REF3450.OUTS
- removed net N$20: R15.2, REF3450.GNDF
- removed net N$5: R3450.OUTF, R4.2
- removed net N$6: R3450.OUTS, R5.2
- removed net VOUT-: U$1.VO-
- net B+INA: now also U$4.VIN+; no longer U$4.VIN-
- net B-INA: now also U$4.VIN-; no longer BAT_PIN.1, U$4.VIN+
- net BATH: now also U1.PD6; no longer U1.PB0
- net BATL: now also U1.PD7; no longer U1.PB1
- net DATAT1: now also U1.PB0; no longer U1.PD6
- net DATAT2: now also U1.PB1; no longer U1.PD7
- net DTR: now also JP1.4; no longer FTDI_PIN.4
- net GND: now also C35.2, JP1.1, R3450.GNDF, REF3450.GNDF, U$1.VO-, U$8.DIO0, U$8.DIO1, U$8.DIO2, U$8.DIO3, U$8.DIO4, U1.PC2, U1.PC3, U1.PD4; no longer BAT_PIN.2, C24.2, FTDI_PIN.1, R15.1, R3.1
- net RX0: now also JP1.3; no longer FTDI_PIN.3
- net TX0: now also JP1.2; no longer FTDI_PIN.2
- net VACS: now also REF3450.OUTF, REF3450.OUTS; no longer R16.1, R17.1
- net VLP5: now also U1.AREF
- net VOUT+: now also C35.1; no longer C24.1
- net VREF5: now also R3450.OUTF, R3450.OUTS; no longer R4.1, R5.1
Other:
- note added: "cambiar por los de 10uF ceramicos de didacticas"
- moved on the sheet: C17, C29

Commit message: placing almost done
Parts:
- removed C34: 2.2uF, rcl:C-EUC1206
- removed JP1: (no value), pinhead:PINHD-1X4/90
- removed U$4: INABB, INA219BB:INABB
- added INA219: INABB, INA219BB:INABB
- added JP2: (no value), pinhead:PINHD-1X4
- added TS3: TERMINAL-TB3, TERMINAL-TB001:TERMINAL-TB3
- C18: value 1uF -> 0.1uF
- C19: value 10uF -> 0.1uF
- renumbered LED3 to BAT-, LED4 to BAT+, U$5 to MCP33121, U1 to ATMEGA328P, U3 to MCP18
Connections:
- net N$16 renamed IN+
- net N$17 renamed IN-
- net N$7 renamed VOMCP18
- new net DATAT3: ATMEGA328P.PD7, C18.1, TS3.2
- net B+INA: now also INA219.VIN+; no longer U$4.VIN+
- net B-INA: now also INA219.VIN-; no longer U$4.VIN-
- net BATH: now also ATMEGA328P.PD5; no longer ATMEGA328P.PD6
- net BATL: now also ATMEGA328P.PD6; no longer ATMEGA328P.PD7
- net DTR: now also JP2.4; no longer JP1.4
- net GND: now also C19.2, INA219.GND, JP2.1, TS1.1, TS2.1, TS3.1; no longer C19.1, C34.1, JP1.1, TS1.3, TS2.3, U$4.GND
- net RX0: now also JP2.3; no longer JP1.3
- net SCL: now also INA219.SCL; no longer U$4.SCL
- net SDA: now also INA219.SDA; no longer U$4.SDA
- net TX0: now also JP2.2; no longer JP1.2
- net VDD33: now also INA219.VCC; no longer U$4.VCC
- net VLP5: now also C19.1, TS1.3, TS2.3, TS3.3; no longer C19.2, C34.2, TS1.1, TS2.1
- net VREF5: no longer C18.1
Other:
- moved on the sheet: C18, C19, C27, C28, C29, C31, C32

Commit message: Finished Placing-Give a review
Parts:
- C2, C3: value cambiar por los de 10uF ceramicos de didacticas -> 10uF
- C23, C6: value 1u -> 10u
Other:
- note added: "1206 10V CERAMICO"
Changed lines of the file:
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@@
 <part name="MCP6002" library="MCP6002-E_MS" deviceset="MCP6002-E/MS" device=""/>
 <part name="LP38692" library="LP38692MP-5.0" deviceset="LP38692MP-5.0" device=""/>
-<part name="C2" library="rcl" library_urn="urn:adsk.eagle:library:334" deviceset="C-EU" device="C1206" package3d_urn="urn:adsk.eagle:package:23618/2" value="cambiar por los de 10uF ceramicos de didacticas"/>
-<part name="C3" library="rcl" library_urn="urn:adsk.eagle:library:334" deviceset="C-EU" device="C1206" package3d_urn="urn:adsk.eagle:package:23618/2" value="cambiar por los de 10uF ceramicos de didacticas"/>
+<part name="C2" library="rcl" library_urn="urn:adsk.eagle:library:334" deviceset="C-EU" device="C1206" package3d_urn="urn:adsk.eagle:package:23618/2" value="10uF "/>
+<part name="C3" library="rcl" library_urn="urn:adsk.eagle:library:334" deviceset="C-EU" device="C1206" package3d_urn="urn:adsk.eagle:package:23618/2" value="10uF "/>
 <part name="2N2222" library="MMBT2222A" deviceset="MMBT2222A" device=""/>
 <part name="R1" library="rcl" library_urn="urn:adsk.eagle:library:334" deviceset="R-EU_" device="R1206" package3d_urn="urn:adsk.eagle:package:23540/2" value="4.7k"/>
 <part name="C4" library="rcl" library_urn="urn:adsk.eagle:library:334" deviceset="C-EU" device="C1206" package3d_urn="urn:adsk.eagle:package:23618/2" value="2.2uF"/>
 <part name="C5" library="rcl" library_urn="urn:adsk.eagle:library:334" deviceset="C-EU" device="C1206" package3d_urn="urn:adsk.eagle:package:23618/2" value="1u"/>
-<part name="C6" library="rcl" library_urn="urn:adsk.eagle:library:334" deviceset="C-EU" device="C1206" package3d_urn="urn:adsk.eagle:package:23618/2" value="1u"/>
+<part name="C6" library="rcl" library_urn="urn:adsk.eagle:library:334" deviceset="C-EU" device="C1206" package3d_urn="urn:adsk.eagle:package:23618/2" value="10u"/>
 <part name="MCP18" library="MCP1501T-18E_SN" deviceset="MCP1501T-18E/SN" device=""/>
 <part name="R6" library="rcl" library_urn="urn:adsk.eagle:library:334" deviceset="R-EU_" device="R0805" package3d_urn="urn:adsk.eagle:package:23553/2" value="10"/>
@@
 <part name="C21" library="rcl" library_urn="urn:adsk.eagle:library:334" deviceset="C-EU" device="C1206" package3d_urn="urn:adsk.eagle:package:23618/2" value="100nF"/>
 <part name="REF3450" library="SOT95P280X145-6N" library_urn="urn:adsk.eagle:library:26233898" deviceset="REF3450" device="" package3d_urn="urn:adsk.eagle:package:26233900/1"/>
-<part name="C23" library="rcl" library_urn="urn:adsk.eagle:library:334" deviceset="C-EU" device="C1206" package3d_urn="urn:adsk.eagle:package:23618/2" value="1u"/>
+<part name="C23" library="rcl" library_urn="urn:adsk.eagle:library:334" deviceset="C-EU" device="C1206" package3d_urn="urn:adsk.eagle:package:23618/2" value="10u"/>
 <part name="U$8" library="XBEE_REG" deviceset="XBEE_REG_MODULE" device=""/>
 <part name="WS1" library="TERMINAL-TB001" deviceset="TERMINAL-TB3" device="" value=""/>
@@
 <wire x1="-129.54" y1="58.42" x2="-129.54" y2="101.6" width="0.1524" layer="97"/>
 <text x="-111.76" y="104.14" size="2.54" layer="97">MODULO DE CARGA</text>
-<text x="-50.8" y="83.82" size="2.1844" layer="97">1206
-10V</text>
+<text x="-50.8" y="68.58" size="2.1844" layer="97">1206
+10V
+CERAMICO</text>
 <text x="35.56" y="76.2" size="2.1844" layer="97">1206</text>
 <text x="45.72" y="71.12" size="2.1844" layer="97">1206
@@
 <instance part="C2" gate="G$1" x="-43.18" y="83.82" smashed="yes">
 <attribute name="NAME" x="-41.656" y="84.201" size="1.778" layer="95"/>
-<attribute name="VALUE" x="-46.736" y="61.341" size="1.778" layer="96"/>
+<attribute name="VALUE" x="-49.276" y="84.201" size="1.778" layer="96"/>
 </instance>
 <instance part="C3" gate="G$1" x="12.7" y="83.82" smashed="yes">

Commit message: pcb ruteada falta plano de tierra
Parts:
- added BATPIN: (no value), pinhead:PINHD-1X2
- added JP1: (no value), pinhead:PINHD-1X3
- renumbered JP2 to FTDI, ON_OFF to ON/OFF, SW2 to RESET, TS1 to T1, TS2 to T2, TS3 to T3, U$1 to POWER-SUPP
Connections:
- net N$2 renamed BASE
- removed net AMOSI: ATMEGA328P.PB3, MCP33121.SDI
- removed net VO: ACS723.VIOUT, C33.1, R11.2
- new net VIN: C33.1, JP1.2, R11.2
- new net VOACS: ACS723.VIOUT, JP1.1
- net B-INA: now also BATPIN.1
- net DATAT1: now also ATMEGA328P.PB1; no longer ATMEGA328P.PB0
- net DATAT2: now also ATMEGA328P.PD7; no longer ATMEGA328P.PB1
- net DATAT3: now also ATMEGA328P.PB0; no longer ATMEGA328P.PD7
- net DATAW1: now also WS1.2; no longer WS1.3
- net DATAW2: now also WS2.2; no longer WS2.3
- net GND: now also ATMEGA328P.PB3, BATPIN.2, JP1.3
- net VLP5: now also MCP33121.SDI, WS1.3, WS2.3; no longer ATMEGA328P.AREF, WS1.2, WS2.2
- net VOUT+: no longer C17.1, C35.1
- net VOW1: now also ATMEGA328P.PC1; no longer ATMEGA328P.PC0
- net VOW2: now also ATMEGA328P.PC0; no longer ATMEGA328P.PC1
- net VSUPPLY: now also C17.1, C35.1, U$8.5V
Other:
- moved on the sheet: ACS723, C15, R10
